File: MH106Enhanced/MH106Enhanced.kicad_pcb (KiCad board)
At the start: 2 copper layers, 22.9 x 53.3 mm, 30 parts, among them J1 Pin 1-20, J2 Pin 21 - 40, J3 5-15V, J4 USB Pins, J5 Conn_01x02, SW1 Bootsel, SW2 Reset, U1 RP2040, U2 TPIC6C595D, U3 TPIC6C595D, U4 TPIC6C595D, U5 AMS1117-3.3, U6 W25Q128JVS

Commit message: Nearly DONE
Parts:
- removed SW1: Bootsel, Button_Switch_SMD:SW_SPST_FSMSM
- removed SW2: Reset, Button_Switch_SMD:SW_SPST_FSMSM
- added C10: 100n, Capacitor_SMD:C_0603_1608Metric_Pad1.08x0.95mm_HandSolder, B.Cu at (101.8, 64.8)
- added C11: 100n, Capacitor_SMD:C_0603_1608Metric_Pad1.08x0.95mm_HandSolder, B.Cu at (101.7, 52.8)
- added C12: 100n, Capacitor_SMD:C_0603_1608Metric_Pad1.08x0.95mm_HandSolder, F.Cu at (102.4, 78.3)
- added C13: 100n, Capacitor_SMD:C_0603_1608Metric_Pad1.08x0.95mm_HandSolder, F.Cu at (102.5, 76.5)
- added C14: 100n, Capacitor_SMD:C_0603_1608Metric_Pad1.08x0.95mm_HandSolder, F.Cu at (102.5, 74.4)
- added C15: 100n, Capacitor_SMD:C_0603_1608Metric_Pad1.08x0.95mm_HandSolder, F.Cu at (102.5, 72.3)
- added C8: 10n, Capacitor_SMD:C_0603_1608Metric_Pad1.08x0.95mm_HandSolder, F.Cu at (99.3, 67.9)
- added C9: 100n, Capacitor_SMD:C_0603_1608Metric_Pad1.08x0.95mm_HandSolder, B.Cu at (101.7, 76.8)
- added J6: I2C, Connector_PinHeader_2.54mm:PinHeader_1x05_P2.54mm_Vertical, F.Cu at (94.6, 77.0)
- added JP1: Reset, Jumper:SolderJumper-2_P1.3mm_Open_RoundedPad1.0x1.5mm, F.Cu at (102.5, 68.4)
- added JP2: Bootsel, Jumper:SolderJumper-2_P1.3mm_Open_RoundedPad1.0x1.5mm, F.Cu at (93.9, 41.4)
- added Q1: BSS138, Package_TO_SOT_SMD:TSOT-23_HandSoldering, B.Cu at (91.9, 76.3)
- added Q2: BSS138, Package_TO_SOT_SMD:TSOT-23_HandSoldering, B.Cu at (91.9, 82.5)
- added R5: 4k7, Resistor_SMD:R_0603_1608Metric_Pad0.98x0.95mm_HandSolder, F.Cu at (97.5, 80.8)
- added R6: 4k7, Resistor_SMD:R_0603_1608Metric_Pad0.98x0.95mm_HandSolder, F.Cu at (100.0, 80.8)
- added U7: ASDMB-xxxMHz, Oscillator:Oscillator_SMD_Abracon_ASDMB-4Pin_2.5x2.0mm, F.Cu at (99.1, 70.1)
- C1, C2, C3, C4: footprint Capacitor_SMD:C_0402_1005Metric -> Capacitor_SMD:C_0603_1608Metric_Pad1.08x0.95mm_HandSolder
- C5, C6: footprint Capacitor_SMD:C_0805_2012Metric -> Capacitor_SMD:C_0603_1608Metric_Pad1.08x0.95mm_HandSolder; moved to B.Cu
- C7: footprint Capacitor_SMD:C_0805_2012Metric -> Capacitor_SMD:C_0603_1608Metric_Pad1.08x0.95mm_HandSolder
- J4: footprint Connector_PinHeader_2.54mm:PinHeader_1x04_P2.54mm_Vertical -> Connector_PinHeader_1.27mm:PinHeader_1x04_P1.27mm_Vertical
- J5: value Conn_01x02 -> Debug; footprint Connector_PinHeader_2.54mm:PinHeader_1x02_P2.54mm_Vertical -> Connector_PinHeader_1.27mm:PinHeader_1x03_P1.27mm_Vertical
- R1, R2: footprint Resistor_SMD:R_0805_2012Metric_Pad1.20x1.40mm_HandSolder -> Resistor_SMD:R_0603_1608Metric_Pad0.98x0.95mm_HandSolder
- R3, R4: footprint Capacitor_SMD:C_0402_1005Metric -> Resistor_SMD:R_0603_1608Metric_Pad0.98x0.95mm_HandSolder
- U6: footprint Package_SO:SOIC-8_3.9x4.9mm_P1.27mm -> Package_SO:SOIC-8W_5.3x5.3mm_P1.27mm
- moved C6 45.3 mm to (92.2, 40.3), turned to 90 degrees
- moved C5 42.6 mm to (94.0, 40.3), turned to 90 degrees
- moved R3 33.0 mm to (94.7, 43.8), turned to 180 degrees
- moved C4 30.9 mm to (103.9, 54.1), turned to 180 degrees
- moved C1 30.1 mm to (98.2, 46.2)
- moved R4 29.9 mm to (94.7, 46.2)
- moved C3 28.6 mm to (102.5, 56.5), turned to 90 degrees
- moved C7 27.6 mm to (105.0, 56.5), turned to 90 degrees
- moved C2 25.4 mm to (103.7, 56.5), turned to 90 degrees
- moved U2 23.8 mm to (99.6, 82.8)
- moved U4 23.3 mm to (99.6, 58.7)
- moved U6 21.2 mm to (99.4, 49.9)
- moved RN1 14.2 mm to (92.6, 50.8)
- moved RN2 13.6 mm to (92.6, 55.2)
- moved RN3 13.0 mm to (92.6, 59.7)
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Connections:
- J1 pad 19: Net-(J1-Pad19) -> STROBE
- J2 pad 3: BCD C/AS 3 -> BCD C/AS 2
- J4 pad 1: 5V -> GND
- J4 pad 4: GND -> 5V
- J5 pad 1: /~{USB_BOOT} -> Net-(J5-Pad1)
- R1 pad 2: Net-(J4-Pad2) -> Net-(J4-Pad3)
- R2 pad 2: Net-(J4-Pad3) -> Net-(J4-Pad2)
- RN6 pad 4: Net-(J1-Pad19) -> STROBE
- RN6 pad 5: STROBE -> STROBE in
- RN6 pad 6: STROBE -> STROBE in
- U1 pad 11: unconnected-(U1-Pad11) -> MC 1
- U1 pad 12: unconnected-(U1-Pad12) -> SST/SSP
- U1 pad 13: unconnected-(U1-Pad13) -> NUL/LAP/LAP
- U1 pad 14: unconnected-(U1-Pad14) -> CHOD.FO/~{NAST}
- U1 pad 15: unconnected-(U1-Pad15) -> PHASE
- U1 pad 16: unconnected-(U1-Pad16) -> STROBE in
- U1 pad 17: unconnected-(U1-Pad17) -> STROBE out
- U1 pad 18: unconnected-(U1-Pad18) -> Shift_SRCK
- U1 pad 20: unconnected-(U1-Pad20) -> XIN
- U1 pad 24: unconnected-(U1-Pad24) -> Net-(J5-Pad1)
- U1 pad 25: unconnected-(U1-Pad25) -> Net-(J5-Pad3)
- U1 pad 27: unconnected-(U1-Pad27) -> Shift_RCK
- U1 pad 28: unconnected-(U1-Pad28) -> Shift_Data
- U1 pad 29: unconnected-(U1-Pad29) -> ~{CAL} out
- U1 pad 31: unconnected-(U1-Pad31) -> SDA
- U1 pad 32: unconnected-(U1-Pad32) -> SCL
- U1 pad 4: unconnected-(U1-Pad4) -> ~{GR}
- U1 pad 5: unconnected-(U1-Pad5) -> EOSC
- U1 pad 6: unconnected-(U1-Pad6) -> Z
- U1 pad 7: unconnected-(U1-Pad7) -> ~{LST}/LSP
- U1 pad 8: unconnected-(U1-Pad8) -> ~{DO}/RY
- U1 pad 9: unconnected-(U1-Pad9) -> MC 0
- U2 pad 1: unconnected-(U2-Pad1) -> +3V3
- U2 pad 10: unconnected-(U2-Pad10) -> Shift_RCK
- U2 pad 11: unconnected-(U2-Pad11) -> BCD A/AS 0
- U2 pad 12: unconnected-(U2-Pad12) -> BCD C/AS 2
- U2 pad 13: unconnected-(U2-Pad13) -> SEG G/NE/AS 4
- U2 pad 14: unconnected-(U2-Pad14) -> ~{ALARM}
- U2 pad 15: unconnected-(U2-Pad15) -> Shift_SRCK
- U2 pad 16: unconnected-(U2-Pad16) -> GND
- U2 pad 2: unconnected-(U2-Pad2) -> Shift_Data
- U2 pad 3: unconnected-(U2-Pad3) -> SEG F/PA/AS 6
- U2 pad 4: unconnected-(U2-Pad4) -> SEG A/SO/AS 5
- U2 pad 5: unconnected-(U2-Pad5) -> BCD D/AS 3
- U2 pad 6: unconnected-(U2-Pad6) -> BCD B/AS 1
- U2 pad 7: unconnected-(U2-Pad7) -> +3V3
- U2 pad 8: unconnected-(U2-Pad8) -> GND
- U2 pad 9: unconnected-(U2-Pad9) -> Net-(U2-Pad9)
- U3 pad 1: unconnected-(U3-Pad1) -> +3V3
- U3 pad 10: unconnected-(U3-Pad10) -> Shift_RCK
- U3 pad 11: unconnected-(U3-Pad11) -> ~{LMS}
- U3 pad 12: unconnected-(U3-Pad12) -> ~{LML}
- U3 pad 13: unconnected-(U3-Pad13) -> ~{LSS}
- U3 pad 14: unconnected-(U3-Pad14) -> ~{LSL}
- U3 pad 15: unconnected-(U3-Pad15) -> Shift_SRCK
- U3 pad 16: unconnected-(U3-Pad16) -> GND
- U3 pad 2: unconnected-(U3-Pad2) -> Net-(U2-Pad9)
- U3 pad 3: unconnected-(U3-Pad3) -> SEG D/PO/AS 10
- U3 pad 4: unconnected-(U3-Pad4) -> SEG C/UT/AS 9
- U3 pad 5: unconnected-(U3-Pad5) -> SEG B/ST/AS 8
- U3 pad 6: unconnected-(U3-Pad6) -> SEG E/CT/AS 7
- U3 pad 7: unconnected-(U3-Pad7) -> +3V3
- U3 pad 8: unconnected-(U3-Pad8) -> GND
- U3 pad 9: unconnected-(U3-Pad9) -> Net-(U3-Pad9)
- U4 pad 1: unconnected-(U4-Pad1) -> +3V3
- U4 pad 10: unconnected-(U4-Pad10) -> Shift_RCK
- U4 pad 11: unconnected-(U4-Pad11) -> ~{DMX 1}
- U4 pad 12: unconnected-(U4-Pad12) -> ~{DMX 3}
- U4 pad 13: unconnected-(U4-Pad13) -> ~{DMX 5}
- U4 pad 14: unconnected-(U4-Pad14) -> ~{DMX 7}
- U4 pad 15: unconnected-(U4-Pad15) -> Shift_SRCK
- U4 pad 16: unconnected-(U4-Pad16) -> GND
- U4 pad 2: unconnected-(U4-Pad2) -> Net-(U3-Pad9)
- U4 pad 3: unconnected-(U4-Pad3) -> ~{DMX 8}
- U4 pad 4: unconnected-(U4-Pad4) -> ~{DMX 6}
- U4 pad 5: unconnected-(U4-Pad5) -> ~{DMX 4}
- U4 pad 6: unconnected-(U4-Pad6) -> ~{DMX 2}
- U4 pad 7: unconnected-(U4-Pad7) -> +3V3
- U4 pad 8: unconnected-(U4-Pad8) -> GND
Routing:
- net GND: track 0.00 -> 196.3 mm, vias 0 -> 8
- net +3V3: track 0.00 -> 159.0 mm, vias 0 -> 7
- net ~{CAL} out: track 0.00 -> 63.2 mm, vias 0 -> 1
- net Net-(U2-Pad9): track 0.00 -> 48.5 mm
- net Shift_RCK: track 0.00 -> 35.2 mm, vias 0 -> 1
- net Net-(U3-Pad9): track 0.00 -> 33.6 mm
- net +1V1: track 0.00 -> 32.4 mm, vias 0 -> 2
- net Shift_SRCK: track 0.00 -> 32.3 mm, vias 0 -> 2
- net SCL: track 0.00 -> 30.6 mm
- net SDA: track 0.00 -> 30.1 mm
- net ~{LSL}: track 0.00 -> 27.6 mm
- net ~{ALARM}: track 0.00 -> 25.5 mm
- net ~{LSS}: track 0.00 -> 23.4 mm
- net ~{DMX 7}: track 0.00 -> 22.1 mm
- net STROBE out: track 0.00 -> 21.9 mm, vias 0 -> 1
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Other:
- board text added: "Bootsel"
- board text added: "Reset"

Commit message: PCB IS DONE
Parts:
- added REF**: OSHW-Logo_5.7x6mm_SilkScreen, Symbol:OSHW-Logo_5.7x6mm_SilkScreen, B.Cu at (101.8, 48.2)
- moved J5 0.20 mm to (96.7, 76.8)
- moved C3 0.08 mm to (102.4, 56.5)
- moved JP1 0.07 mm to (102.4, 68.3)
- moved JP2 0.05 mm to (93.8, 41.4)
Routing:
- net Shift_RCK: track 35.2 -> 46.6 mm, vias 1 -> 2
- net +1V1: track 32.4 -> 28.4 mm
- net +3V3: track 159.0 -> 162.6 mm
- net Shift_Data: track 17.0 -> 18.0 mm
- net SEG D/PO/AS 10: track 10.5 -> 11.0 mm
- net GND: track 196.3 -> 196.8 mm
- added copper zone on B.Cu, net GND
- added copper zone on F.Cu, net GND
Other:
- board text added: "JLCJLCJLCJLC"
- board text added: "Michael's Lab 02-2023 MH106 Clone RP2040"
- board text removed: "Michael's Lab 02-2023"
