File: MH106Enhanced/MH106Enhanced.kicad_sch (KiCad schematic)
At the start: 44 parts, among them J1 Pin 1-20, J2 Pin 21 - 40, J3 5-15V, J4 USB Pins, J5 Debug, J6 I2C, Q1 BSS138, Q2 BSS138, U1 RP2040, U2 TPIC6C595D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

Commit message: PCB IS DONE
Connections:
- net Shift_Data: now also U1.28 (GPIO17); no longer U1.27 (GPIO16)
- net Shift_RCK: now also U1.27 (GPIO16); no longer U1.28 (GPIO17)
Changed lines of the file:
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@@
     (stroke (width 0) (type default) (color 0 0 0 0))
   )
-  (wire (pts (xy 137.16 147.32) (xy 142.24 147.32))
-    (stroke (width 0) (type default) (color 0 0 0 0))
-  )
   (wire (pts (xy 274.32 184.15) (xy 274.32 185.42))
     (stroke (width 0) (type default) (color 0 0 0 0))
@@
     (stroke (width 0) (type default) (color 0 0 0 0))
   )
-  (wire (pts (xy 137.16 144.78) (xy 142.24 144.78))
-    (stroke (width 0) (type default) (color 0 0 0 0))
-  )
   (wire (pts (xy 393.7 104.14) (xy 393.7 106.68))
     (stroke (width 0) (type default) (color 0 0 0 0))
@@
     (stroke (width 0) (type default) (color 0 0 0 0))
   )
+  (wire (pts (xy 137.16 147.32) (xy 142.24 147.32))
+    (stroke (width 0) (type default) (color 0 0 0 0))
+  )
   (wire (pts (xy 220.98 200.66) (xy 246.38 200.66))
     (stroke (width 0) (type default) (color 0 0 0 0))
@@
     (stroke (width 0) (type default) (color 0 0 0 0))
   )
+  (wire (pts (xy 137.16 144.78) (xy 142.24 144.78))
+    (stroke (width 0) (type default) (color 0 0 0 0))
+  )
   (wire (pts (xy 316.23 95.25) (xy 316.23 96.52))
     (stroke (width 0) (type default) (color 0 0 0 0))
@@
     )
   )
-  (global_label "Shift_Data" (shape input) (at 142.24 144.78 0) (fields_autoplaced)
+  (global_label "Shift_Data" (shape input) (at 142.24 147.32 0) (fields_autoplaced)
     (effects (font (size 1.27 1.27)) (justify left))
-    (property "Intersheet References" "${INTERSHEET_REFS}" (id 0) (at 154.3293 144.8594 0)
+    (property "Intersheet References" "${INTERSHEET_REFS}" (id 0) (at 154.3293 147.3994 0)
       (effects (font (size 1.27 1.27)) (justify left) hide)
     )
@@
     )
   )
-  (global_label "Shift_RCK" (shape input) (at 142.24 147.32 0) (fields_autoplaced)
+  (global_label "Shift_RCK" (shape input) (at 142.24 144.78 0) (fields_autoplaced)
     (effects (font (size 1.27 1.27)) (justify left))
-    (property "Intersheet References" "${INTERSHEET_REFS}" (id 0) (at 153.8455 147.3994 0)
+    (property "Intersheet References" "${INTERSHEET_REFS}" (id 0) (at 153.8455 144.8594 0)
       (effects (font (size 1.27 1.27)) (justify left) hide)
     )
@@
     (pin "2")
   )
+  (symbol (lib_id "Graphic:Logo_Open_Hardware_Large") (at 388.62 238.76 0) (unit 1)
+    (in_bom yes) (on_board yes) (fields_autoplaced)
+    (property "Reference" "#LOGO1" (id 0) (at 388.62 226.06 0)
+      (effects (font (size 1.27 1.27)) hide)
+    )
+    (property "Value" "Logo_Open_Hardware_Large" (id 1) (at 388.62 248.92 0)
+      (effects (font (size 1.27 1.27)) hide)
+    )
+    (property "Footprint" "" (id 2) (at 388.62 238.76 0)
+      (effects (font (size 1.27 1.27)) hide)
+    )
+    (property "Datasheet" "~" (id 3) (at 388.62 238.76 0)
+      (effects (font (size 1.27 1.27)) hide)
+    )
+  )
   (symbol (lib_id "Device:C") (at 400.05 129.54 0) (unit 1)
     (in_bom yes) (on_board yes)
@@
   )
   (symbol_instances
+    (path "/1c141c88-f674-43b1-95d3-d570287fd457"
+      (reference "#LOGO1") (unit 1) (value "Logo_Open_Hardware_Large") (footprint "")
+    )
     (path "/fea1255a-73c6-40a3-a782-b0dc771ccc0a"
       (reference "#PWR01") (unit 1) (value "+3V3") (footprint "")
